Commit message: 18/10/2023

File: assignment2/urdf/closedChain.urdf.xacro (robot description, xacro)
@@ -26,5 +26,5 @@
   <link name="bo">
     <visual>
-    <origin xyz="0.0 0.0 0.025" rpy="0.0 0.0 0.0"/>
+    <origin xyz="0.0 0.0 0.025" rpy="0.0 0.0 150"/>
     <geometry>
       <cylinder radius="0.025" length="0.05"/>
